File: Capteur_courant_IoT/_autosave-Capteur_courant_IoT.kicad_pcb (KiCad board)
At the start: 2 copper layers, 48 parts, among them J2 Conn_01x04_Socket, J4 Conn_01x04_Socket, J5 USB4105-GF-A, Q1 SS8050, Q2 SS8050, Q3 FDN340P, Q5 FDN340P, U1 CP2102N-Axx-xQFN28, U2 ESP32-WROOM-32E, U3 TPS62162DSG, U4 ADS1015IDGS

Commit message: correction des points évoqués
Parts:
- removed D1, D10, D9: ESDZL5-1F4, Diode_SMD:D_0201_0603Metric
- removed D3, D7: SP0503BAHT, Package_TO_SOT_SMD:SOT-143
- added C11: C, Capacitor_SMD:C_0603_1608Metric, F.Cu at (147.7, 181.5)
- added D12: ESDZL2012MX4T5G, Diode_SMD:D_0201_0603Metric, F.Cu at (140.7, 171.5)
- added D4: LED_B, LED_SMD:LED_0805_2012Metric, F.Cu at (141.5, 175.9)
- added D5: LED_G, LED_SMD:LED_0805_2012Metric, F.Cu at (141.5, 178.9)
- added D6: LED_R, LED_SMD:LED_0805_2012Metric, F.Cu at (141.5, 181.9)
- added R15: 0R, Resistor_SMD:R_0805_2012Metric, F.Cu at (147.9, 175.8)
- added R20: R, Resistor_SMD:R_0805_2012Metric, F.Cu at (147.9, 178.8)
- added U5: USBLC6-2SC6, Package_TO_SOT_SMD:SOT-23-6, F.Cu at (150.3, 168.8)
- added U6: D3V3XA4B10LP, Package_DFN_QFN:Diodes_UDFN-10_1.0x2.5mm_P0.5mm, F.Cu at (141.0, 168.6)
- added U7: D3V3XA4B10LP, Package_DFN_QFN:Diodes_UDFN-10_1.0x2.5mm_P0.5mm, F.Cu at (144.2, 168.6)
- R4: value 22.1k -> 22k
- R5: value 47.5K -> 47k
Connections:
- C3 pad 1: GND -> /ESP32/GPIO34
- C3 pad 2: /ESP32/GPIO34 -> GND
- C4 pad 1: GND -> /ESP32/GPIO35
- C4 pad 2: /ESP32/GPIO35 -> GND
- C5 pad 1: GND -> /ESP32/EN
- C5 pad 2: /ESP32/EN -> GND
- U1 pad 4: /dp -> Net-(U1-D+)
- U1 pad 5: /dn -> Net-(U1-D-)
- U4 pad 4: /ESP32/AINpositif -> Net-(U4-AIN0)
