File: Capteur_courant_IoT/Alimentation.kicad_sch (KiCad schematic)
At the start: 11 parts, among them Q3 FDN340P, Q4 FQP27P06, U3 TPS62162DSG

Commit message: correction des points évoqués
Parts:
- removed Q4: FQP27P06, Package_TO_SOT_THT:TO-220-3_Vertical, symbol Transistor_FET:FQP27P06
- added Q5: FDN340P, Package_TO_SOT_SMD:SOT-23, symbol Transistor_FET:FDN340P
- C8, C9: footprint (none) -> Capacitor_SMD:C_0603_1608Metric
- D8: value D_Zener -> diode 5.1V
- L1: value 2.2µH -> VLS4012ET-2R2M
- R11, R12, R14: footprint (none) -> Resistor_SMD:R_0805_2012Metric
Connections:
- net Vin: now also Q5.3 (D)
- net at D2.2 (A), D8.1 (K), Q3.1 (G)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: now also Q5.2 (S)
- net at D8.2 (A), R14.1: now also Q5.1 (G)
Changed lines of the file:
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@@
 			)
 		)
-		(property "Footprint" ""
+		(property "Footprint" "Capacitor_SMD:C_0603_1608Metric"
 			(at 147.0152 111.76 0)
 			(effects
@@
 			)
 		)
-		(property "Value" "D_Zener"
+		(property "Value" "diode 5.1V"
 			(at 53.34 71.1199 90)
 			(effects
@@
 			)
 		)
-		(property "Footprint" ""
+		(property "Footprint" "Resistor_SMD:R_0805_2012Metric"
 			(at 195.072 120.65 90)
 			(effects
@@
 	)
 	(symbol
+		(lib_id "Transistor_FET:FDN340P")
+		(at 38.1 66.04 90)
+		(unit 1)
+		(exclude_from_sim no)
+		(in_bom yes)
+		(on_board yes)
+		(dnp no)
+		(fields_autoplaced yes)
+		(property "Reference" "Q5"
+			(at 36.8299 59.69 0)
+			(effects
+				(font
+					(size 1.27 1.27)
+				)
+				(justify left)
+			)
+		)
+		(property "Value" "FDN340P"
+			(at 39.3699 59.69 0)
+			(effects
+				(font
+					(size 1.27 1.27)
+				)
+				(justify left)
+			)
+		)
+		(property "Footprint" "Package_TO_SOT_SMD:SOT-23"
+			(at 40.005 60.96 0)
+			(effects
+				(font
+					(size 1.27 1.27)
+					(italic yes)
+				)
+				(justify left)
+				(hide yes)
+			)
+		)
+		(property "Datasheet" "https://www.onsemi.com/pub/Collateral/FDN340P-D.PDF"
+			(at 41.91 60.96 0)
+			(effects
+				(font
+					(size 1.27 1.27)
+				)
+				(justify left)
+				(hide yes)
+			)
+		)
+		(property "Description" "-2A Id, -20V Vds, P-Channel MOSFET, 70mOhm Ron, SOT-23"
+			(at 38.1 66.04 0)
+			(effects
+				(font
+					(size 1.27 1.27)
+				)
+				(hide yes)
+			)
+		)
+		(pin "1"
+		)
+		(pin "3"
+		)
+		(pin "2"
+		)
+		(instances
+			(project "Capteur_courant_IoT"
+				(path "/9ec92dd4-bf7f-4382-b228-27fa2b950a1e/b6506b61-f6f9-4e50-8bb0-94b375784be5"
+					(reference "Q5")
+					(unit 1)
+				)
+			)
+		)
+	)
+	(symbol
 		(lib_id "power:VBUS")
 		(at 63.5 99.06 0)
@@
 			)
 		)
-		(property "Footprint" ""
+		(property "Footprint" "Resistor_SMD:R_0805_2012Metric"
 			(at 36.322 82.55 90)
 			(effects
@@
 			)
 		)
-		(property "Footprint" ""
+		(property "Footprint" "Resistor_SMD:R_0805_2012Metric"
 			(at 99.822 82.55 90)
 			(effects
@@
 	)
 	(symbol
-		(lib_id "Transistor_FET:FQP27P06")
-		(at 38.1 66.04 90)
-		(unit 1)
-		(exclude_from_sim no)
-		(in_bom yes)
-		(on_board yes)
-		(dnp no)
-		(fields_autoplaced yes)
-		(property "Reference" "Q4"
-			(at 38.1 57.15 90)
-			(effects
-				(font
-					(size 1.27 1.27)
-				)
-			)
-		)
-		(property "Value" "FQP27P06"
-			(at 38.1 59.69 90)
-			(effects
-				(font
-					(size 1.27 1.27)
-				)
-			)
-		)
-		(property "Footprint" "Package_TO_SOT_THT:TO-220-3_Vertical"
-			(at 40.005 60.96 0)
-			(effects
-				(font
-					(size 1.27 1.27)
-					(italic yes)
-				)
-				(justify left)
-				(hide yes)
-			)
-		)
-		(property "Datasheet" "https://www.onsemi.com/pub/Collateral/FQP27P06-D.PDF"
-			(at 41.91 60.96 0)
-			(effects
-				(font
-					(size 1.27 1.27)
-				)
-				(justify left)
-				(hide yes)
-			)
-		)
-		(property "Description" "-27A Id, -60V Vds, QFET P-Channel MOSFET, TO-220"
-			(at 38.1 66.04 0)
-			(effects
-				(font
-					(size 1.27 1.27)
-				)
-				(hide yes)
-			)
-		)
-		(pin "2"
-		)
-		(pin "3"
-		)
-		(pin "1"
-		)
-		(instances
-			(project ""
-				(path "/9ec92dd4-bf7f-4382-b228-27fa2b950a1e/b6506b61-f6f9-4e50-8bb0-94b375784be5"
-					(reference "Q4")
-					(unit 1)
-				)
-			)
-		)
-	)
-	(symbol
 		(lib_id "power:GND")
 		(at 215.9 114.3 0)
@@
 			)
 		)
-		(property "Footprint" ""
+		(property "Footprint" "Capacitor_SMD:C_0603_1608Metric"
 			(at 216.8652 111.76 0)
 			(effects
@@
 			)
 		)
-		(property "Value" "2.2µH"
+		(property "Value" "VLS4012ET-2R2M"
 			(at 191.7699 93.98 0)
 			(effects

Commit message: V100
Parts:
- removed D8: diode 5.1V, symbol Device:D_Zener
- removed L1: VLS4012ET-2R2M, symbol Device:L
- added D1: BZT52Bxx, Diode_SMD:D_SOD-123, symbol Diode:BZT52Bxx
- added L1: LQH2HPZ2R2MJRL, Library_iot:IND_LQH2HPZ2R2MJRL, symbol library_perso:LQH2HPZ2R2MJRL
- C8, C9: footprint Capacitor_SMD:C_0603_1608Metric -> Capacitor_SMD:C_0805_2012Metric
- D2: value D_Schottky_inversion -> BAT54WS; footprint (none) -> Diode_SMD:D_SOD-323
Connections:
- net +3.3V: now also L1.2
- net at D2.2 (A), Q3.1 (G), Q5.2 (S)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: now also D1.1 (K)
- net at Q5.1 (G), R14.1: now also D1.2 (A)
- net at U3.7 (SW): now also L1.1
Other:
- moved on the sheet: D2
