File: Capteur_courant_IoT/Capteur_courant_IoT.kicad_pcb (KiCad board)
At the start: 2 copper layers, 48 parts, among them J2 Conn_01x04_Socket, J4 Conn_01x04_Socket, J5 USB4105-GF-A, Q1 SS8050, Q2 SS8050, Q3 FDN340P, Q5 FDN340P, U1 CP2102N-Axx-xQFN28, U2 ESP32-WROOM-32E, U3 TPS62162DSG, U4 ADS1015IDGS

Commit message: V100
Parts:
- removed D10, D9: ESDZL5-1F4, Diode_SMD:D_0201_0603Metric
- removed R17, R19: 10K, Resistor_SMD:R_0805_2012Metric
- added C11: C, Capacitor_SMD:C_0805_2012Metric, F.Cu at (164.3, 88.7)
- added D12: ESDZL2012MX4T5G, Diode_SMD:D_0201_0603Metric, F.Cu at (163.6, 81.9)
- added D2: BAT54WS, Diode_SMD:D_SOD-323, F.Cu at (145.2, 120.0)
- added D4: LED_B, LED_SMD:LED_0805_2012Metric, F.Cu at (145.2, 101.2)
- added D5: LED_G, LED_SMD:LED_0805_2012Metric, F.Cu at (142.5, 101.2)
- added D6: LED_R, LED_SMD:LED_0805_2012Metric, F.Cu at (148.0, 101.3)
- added H1: MountingHole_Pad, MountingHole:MountingHole_3.2mm_M3_DIN965_Pad, F.Cu at (161.5, 95.0)
- added H2: MountingHole_Pad, MountingHole:MountingHole_3.2mm_M3_DIN965_Pad, F.Cu at (127.0, 95.0)
- added H3: MountingHole_Pad, MountingHole:MountingHole_3.2mm_M3_DIN965_Pad, F.Cu at (127.0, 123.0)
- added J1: ED555/2DS, Library_iot:CONN_ED555&slash_2DS_OST, F.Cu at (161.5, 120.6)
- added J3: ED555/2DS, Library_iot:CONN_ED555&slash_2DS_OST, F.Cu at (161.4, 75.6)
- added L1: LQH2HPZ2R2MJRL, Library_iot:IND_LQH2HPZ2R2MJRL, F.Cu at (145.9, 107.5)
- added R15: 0R, Resistor_SMD:R_0805_2012Metric, F.Cu at (156.5, 74.7)
- added R20: R, Resistor_SMD:R_0805_2012Metric, F.Cu at (164.3, 85.0)
- added U5: USBLC6-2SC6, Package_TO_SOT_SMD:SOT-23-6, F.Cu at (153.8, 109.6)
- added U6: D3V3XA4B10LP, Package_DFN_QFN:Diodes_UDFN-10_1.0x2.5mm_P0.5mm, F.Cu at (125.8, 104.8)
- added U7: D3V3XA4B10LP, Package_DFN_QFN:Diodes_UDFN-10_1.0x2.5mm_P0.5mm, F.Cu at (145.8, 95.5)
- C1, C10, C2, C3, C4, C5, C6, C7, C8, C9: footprint Capacitor_SMD:C_0603_1608Metric -> Capacitor_SMD:C_0805_2012Metric
- D1: value ESDZL5-1F4 -> BZT52Bxx; footprint Diode_SMD:D_0201_0603Metric -> Diode_SMD:D_SOD-123
- D3, D7: value SP0503BAHT -> BAT54WS; footprint Package_TO_SOT_SMD:SOT-143 -> Diode_SMD:D_SOD-323
- R3: value 10K -> 0R
- R4: value 22.1k -> 22k
- R5: value 47.5K -> 47k
- U2: footprint RF_Module:ESP32-WROOM-32D -> RF_Module:ESP32-WROOM-32E
- moved J2 119.7 mm to (142.2, 96.0), turned to -90 degrees
- moved S3 110.2 mm to (137.6, 103.5), turned to -90 degrees
- moved S2 102.7 mm to (130.7, 103.5), turned to 90 degrees
- moved S1 99.1 mm to (126.5, 85.2), turned to 90 degrees
- moved J4 96.5 mm to (126.0, 110.2)
- moved U4 95.8 mm to (160.8, 86.2), turned to -90 degrees
- moved D11 75.3 mm to (156.9, 123.7), turned to 90 degrees
- moved J5 71.1 mm to (162.6, 112.8), turned to 90 degrees
- moved Q2 70.4 mm to (155.2, 96.3), turned to 90 degrees
- moved C4 69.7 mm to (138.0, 111.2), turned to -90 degrees
- moved C2 68.6 mm to (125.7, 75.5), turned to 90 degrees
- moved D1 66.6 mm to (148.2, 123.4)
- moved C1 66.3 mm to (128.5, 75.5), turned to 90 degrees
- moved Q1 64.6 mm to (151.4, 96.3), turned to 90 degrees
- moved C5 64.3 mm to (124.3, 79.1), turned to -90 degrees
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Connections:
- net /ESP32/RXD0 renamed /ESP32/RXD0_cp2102 -- TXD0_ESP32
- net /ESP32/TXD0 renamed /ESP32/TXD0_cp2102 -- RXD0_ESP32
- C3 pad 1: GND -> /ESP32/GPIO34
- C3 pad 2: /ESP32/GPIO34 -> GND
- C4 pad 1: GND -> /ESP32/GPIO35
- C4 pad 2: /ESP32/GPIO35 -> GND
- C5 pad 1: GND -> Net-(D3-K)
- C5 pad 2: /ESP32/EN -> GND
- D1 pad 1: /dn -> Net-(D1-K)
- D1 pad 2: GND -> Net-(D1-A)
- D3 pad 1: GND -> Net-(D3-K)
- D3 pad 2: /ESP32/SDA -> /ESP32/EN
- D7 pad 1: GND -> Net-(D7-K)
- D7 pad 2: /ESP32/SDA -> /ESP32/EN
- J2 pad 3: GND -> +3.3V
- J2 pad 4: +3.3V -> GND
- J4 pad 3: GND -> +3.3V
- J4 pad 4: +3.3V -> GND
- Q1 pad 3: /ESP32/EN -> Net-(D7-K)
- Q3 pad 1: Net-(D2-A) -> Net-(D1-K)
- Q5 pad 1: Net-(D8-A) -> Net-(D1-A)
- Q5 pad 2: Net-(D2-A) -> Net-(D1-K)
- R11 pad 1: Net-(D2-A) -> Net-(D1-K)
- R14 pad 1: Net-(D8-A) -> Net-(D1-A)
- R16 pad 2: Net-(R16-Pad2) -> /ESP32/GPIO34
- R18 pad 2: Net-(R18-Pad2) -> /ESP32/GPIO35
- R3 pad 1: Net-(R3-Pad1) -> Net-(U4-AIN3)
- R3 pad 2: /ESP32/EN -> /ESP32/AINnégatif
- S1 pad 3: Net-(R3-Pad1) -> Net-(D3-K)
- S1 pad 4: Net-(R3-Pad1) -> Net-(D3-K)
- S2 pad 3: Net-(R16-Pad2) -> /ESP32/GPIO34
- S2 pad 4: Net-(R16-Pad2) -> /ESP32/GPIO34
- S3 pad 3: Net-(R18-Pad2) -> /ESP32/GPIO35
- S3 pad 4: Net-(R18-Pad2) -> /ESP32/GPIO35
- U1 pad 4: /dp -> Net-(U1-D+)
- U1 pad 5: /dn -> Net-(U1-D-)
- U4 pad 4: /ESP32/AINpositif -> Net-(U4-AIN0)
- U4 pad 7: /ESP32/AINnégatif -> Net-(U4-AIN3)
Routing:
- net GND: track 0.00 -> 97.4 mm, vias 0 -> 157
- net /ESP32/SCL: track 0.00 -> 83.6 mm, vias 0 -> 2
- net /ESP32/SDA: track 0.00 -> 79.2 mm, vias 0 -> 7
- net +3.3V: track 0.00 -> 63.7 mm, vias 0 -> 16
- net /ESP32/GPIO35: track 0.00 -> 43.1 mm, vias 0 -> 1
- net /ESP32/GPIO34: track 0.00 -> 36.6 mm, vias 0 -> 1
- net Net-(D7-K): track 0.00 -> 35.4 mm, vias 0 -> 2
- net /ESP32/GPIO32: track 0.00 -> 31.7 mm, vias 0 -> 2
- net /ESP32/GPIO33: track 0.00 -> 31.3 mm, vias 0 -> 2
- net /ESP32/GPIO27: track 0.00 -> 28.9 mm, vias 0 -> 2
- net /ESP32/RXD0_cp2102 -- TXD0_ESP32: track 0.00 -> 27.7 mm
- net VBUS: track 0.00 -> 26.7 mm, vias 0 -> 4
- net /ESP32/TXD0_cp2102 -- RXD0_ESP32: track 0.00 -> 25.8 mm
- net Net-(D6-K): track 0.00 -> 22.7 mm, vias 0 -> 2
- net Net-(D5-K): track 0.00 -> 22.4 mm, vias 0 -> 2
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- added copper zone on F.Cu, net +3.3V
- added copper zone on In2.Cu, net +3.3V
- added copper zone on F.Cu, net +5V
- added copper zone on B.Cu, net GND
- added copper zone on F.Cu, net GND
- added copper zone on In1.Cu, net GND
Other:
- board outline added: 42.5 x 53.4 mm
- copper layers 2 -> 4
- board text added: "LE CLICK 23/07/2025 IF-C100 Khalil Bendjelal"
