File: Capteur_courant_IoT/USB.kicad_sch (KiCad schematic)
At the start: 12 parts, among them Q1 SS8050, Q2 SS8050, U1 CP2102N-Axx-xQFN28

Commit message: correction des points évoqués
Parts:
- removed D1: SP0503BAHT, Package_TO_SOT_SMD:SOT-143, symbol Power_Protection:SP0503BAHT
- removed R3: 10K, symbol Device:R
- added U5: USBLC6-2SC6, Package_TO_SOT_SMD:SOT-23-6, symbol Power_Protection:USBLC6-2SC6
- C6, C7: footprint (none) -> Capacitor_SMD:C_0603_1608Metric
- R1, R2, R6: footprint (none) -> Resistor_SMD:R_0805_2012Metric
- R4: value 22.1k -> 22k; footprint (none) -> Resistor_SMD:R_0805_2012Metric
- R5: value 47.5K -> 47k; footprint (none) -> Resistor_SMD:R_0805_2012Metric
Connections:
- net D+: now also U5.1 (I/O1); no longer U1.4 (D+)
- net D-: now also U5.3 (I/O2); no longer U1.5 (D-)
- net GND: now also U5.2 (GND)
- net VBUS: now also U5.5 (VBUS)
- new net: U1.5 (D-), U5.4 (I/O2)
- new net: U1.4 (D+), U5.6 (I/O1)
- no-connect marks 15 -> 16
Other:
- moved on the sheet: C6, C7

Commit message: V100
Parts:
- added D7: BAT54WS, Diode_SMD:D_SOD-323, symbol Device:D_Schottky
- C6, C7: footprint Capacitor_SMD:C_0603_1608Metric -> Capacitor_SMD:C_0805_2012Metric
Connections:
- net EN: now also D7.2 (A); no longer Q1.3 (C)
- new net: D7.1 (K), Q1.3 (C)
Changed lines of the file:
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@@
+	(wire
+		(pts
+			(xy 251.46 64.77) (xy 254 64.77)
+		)
+		(stroke
+			(width 0)
+			(type default)
+		)
+	)
 	(wire
 		(pts
@@
 	(wire
 		(pts
-			(xy 241.3 64.77) (xy 254 64.77)
+			(xy 241.3 64.77) (xy 243.84 64.77)
 		)
 		(stroke
@@
 			)
 		)
-		(property "Footprint" "Capacitor_SMD:C_0603_1608Metric"
+		(property "Footprint" "Capacitor_SMD:C_0805_2012Metric"
 			(at 115.2652 35.56 0)
 			(effects
@@
 	)
 	(symbol
+		(lib_id "Device:D_Schottky")
+		(at 247.65 64.77 0)
+		(unit 1)
+		(exclude_from_sim no)
+		(in_bom yes)
+		(on_board yes)
+		(dnp no)
+		(property "Reference" "D7"
+			(at 247.65 57.404 0)
+			(effects
+				(font
+					(size 1.27 1.27)
+				)
+			)
+		)
+		(property "Value" "BAT54WS"
+			(at 247.65 60.198 0)
+			(effects
+				(font
+					(size 1.27 1.27)
+				)
+			)
+		)
+		(property "Footprint" "Diode_SMD:D_SOD-323"
+			(at 247.65 64.77 0)
+			(effects
+				(font
+					(size 1.27 1.27)
+				)
+				(hide yes)
+			)
+		)
+		(property "Datasheet" "~"
+			(at 247.65 64.77 0)
+			(effects
+				(font
+					(size 1.27 1.27)
+				)
+				(hide yes)
+			)
+		)
+		(property "Description" "Schottky diode"
+			(at 247.65 64.77 0)
+			(effects
+				(font
+					(size 1.27 1.27)
+				)
+				(hide yes)
+			)
+		)
+		(pin "1"
+		)
+		(pin "2"
+		)
+		(instances
+			(project "Capteur_courant_IoT"
+				(path "/9ec92dd4-bf7f-4382-b228-27fa2b950a1e/5dcc9638-5970-4d96-845c-272768bc2ec4"
+					(reference "D7")
+					(unit 1)
+				)
+			)
+		)
+	)
+	(symbol
 		(lib_id "Interface_USB:CP2102N-Axx-xQFN28")
 		(at 142.24 109.22 0)
@@
 			)
 		)
-		(property "Footprint" "Capacitor_SMD:C_0603_1608Metric"
+		(property "Footprint" "Capacitor_SMD:C_0805_2012Metric"
 			(at 127.9652 35.56 0)
 			(effects
